File: pcb/messenger/messenger.kicad_pcb (KiCad board)
At the start: 4 copper layers, 68 x 73.5 mm, 85 parts, among them J1 USB_C_Receptacle_USB2.0_16P, J2 Battery, J3 Conn_Coaxial, J4 Display Connector, J5 Conn_Coaxial, Q1_Xtal1 32.0MHz, SW1 BOOT, SW2 EN, U1 DMG3415U-7, U10 W25Q128JVS, U12 BBQ10KBD, U13 TCA8418RTWR, U14 24AA32AF-I_MS, U17 MAX17048G+T10, U2 ESP32-S3, U3 SX1262IMLTRT, U4 USBLC6-2SC6, U5 MCP73831-2-OT, U6 BGS12WN6E6327, U7 TLV76733DRVx, U8 DMG3415U-7, U9 DMG3415U-7, X1 40MHz

Commit message: pcb fixes
Parts:
- removed R8: 5.1k, Resistor_SMD:R_0603_1608Metric
- added R21: 10, Resistor_SMD:R_0603_1608Metric, F.Cu at (155.8, 69.0)
Connections:
- J4 pad 3: Net-(J4-Pin_3) -> GND
- J4 pad 4: Net-(J4-Pin_3) -> GND
- U9 pad 3: Net-(J4-Pin_20) -> Net-(U9-D)
Routing:
- net Net-(J4-Pin_3): track 10.7 -> 0.00 mm
- net Net-(J4-Pin_20): track 8.48 -> 3.58 mm
- net Net-(U9-D): track 0.00 -> 3.47 mm
- net GND: vias 433 -> 142
