File: pcb/messenger/messenger.kicad_pcb (KiCad board)
At the start: 4 copper layers, 68 x 73.5 mm, 85 parts, among them J1 USB_C_Receptacle_USB2.0_16P, J2 Battery, J3 Conn_Coaxial, J4 Display Connector, J5 Conn_Coaxial, Q1_Xtal1 32.0MHz, SW1 BOOT, SW2 EN, U1 DMG3415U-7, U10 W25Q128JVS, U12 BBQ10KBD, U13 TCA8418RTWR, U14 24AA32AF-I_MS, U17 MAX17048G+T10, U2 ESP32-S3, U3 SX1262IMLTRT, U4 USBLC6-2SC6, U5 MCP73831-2-OT, U6 BGS12WN6E6327, U7 TLV76733DRVx, U8 DMG3415U-7, U9 DMG3415U-7, X1 40MHz

Commit message: still dont work
Parts:
- removed R8: 5.1k, Resistor_SMD:R_0603_1608Metric
- removed U6: BGS12WN6E6327, Package_LGA:Infineon_PG-TSNP-6-10_0.7x1.1mm_0.7x1.1mm_P0.4mm
- added C29: 10uF, Capacitor_SMD:C_0603_1608Metric, F.Cu at (164.4, 113.2)
- added C30: 22uF, Capacitor_SMD:C_0603_1608Metric, F.Cu at (154.9, 110.9)
- added R21: 10, Resistor_SMD:R_0603_1608Metric, F.Cu at (156.6, 69.3)
- added R22: 100R, Resistor_SMD:R_0402_1005Metric, F.Cu at (168.5, 59.8)
- added U15: TLV76733DRVx, Package_SON:WSON-6-1EP_2x2mm_P0.65mm_EP1x1.6mm_ThermalVias, F.Cu at (159.3, 111.4)
- added U18: PE4259, PE4259:SC-70-6_PSM, F.Cu at (171.5, 60.9)
- J5: footprint Connector_Coaxial:SMA_Amphenol_901-143_Horizontal -> Connector_Coaxial:U.FL_Molex_MCRF_73412-0110_Vertical
- moved R18 25.9 mm to (159.4, 114.3), turned to 180 degrees
- moved C8 15.6 mm to (141.7, 71.3), turned to 90 degrees
- moved L1 10.7 mm to (122.1, 59.5)
- moved C20 10.5 mm to (171.9, 86.6), turned to 90 degrees
- moved C19 8.48 mm to (170.5, 86.3), turned to 90 degrees
- moved R16 5.43 mm to (174.2, 59.8), turned to 0 degrees
- moved C26 5.40 mm to (174.1, 58.7), turned to 0 degrees
- moved C25 5.28 mm to (168.5, 58.7)
- moved C27 2.83 mm to (171.5, 56.7)
- moved J5 2.58 mm to (171.4, 51.5)
- moved R4 2.43 mm to (126.3, 116.2), turned to -90 degrees
- moved R11 0.71 mm to (119.0, 56.6), turned to 90 degrees
Connections:
- ATGM336H1 pad 5: GPS_ON/OFF -> unconnected-(ATGM336H1-ON/OFF-Pad5)
- ATGM336H1 pad 8: +3V3 -> +3V3_2
- C19 pad 1: +3V3 -> +3V3_2
- C20 pad 1: +3V3 -> +3V3_2
- J4 pad 2: +3V3 -> +3V3_2
- J4 pad 3: Net-(J4-Pin_3) -> GND
- J4 pad 4: Net-(J4-Pin_3) -> GND
- R10 pad 1: +3V3 -> +3V3_2
- R13 pad 1: +3V3 -> +3V3_2
- R15 pad 1: +3V3 -> +3V3_2
- R18 pad 1: GPS_ON/OFF -> LDO_EN
- R9 pad 1: +3V3 -> +3V3_2
- U1 pad 2: +3V3 -> +3V3_2
- U13 pad 21: +3V3 -> +3V3_2
- U14 pad 8: +3V3 -> +3V3_2
- U17 pad 3: unconnected-(U17-VDD-Pad3) -> +3V3
- U2 pad 19: LORA_DIO1 -> LDO_EN
- U2 pad 22: GPS_ON/OFF -> LORA_DIO1
- U9 pad 2: +3V3 -> +3V3_2
- U9 pad 3: Net-(J4-Pin_20) -> Net-(U9-D)
Routing:
- net +3V3_2: track 0.00 -> 136.3 mm, vias 0 -> 6
- net LDO_EN: track 0.00 -> 76.0 mm, vias 0 -> 4
- net GPS_ON/OFF: track 73.0 -> 0.00 mm, vias 2 -> 0
- net VCC: track 14.7 -> 52.8 mm
- net +3V3: track 74.0 -> 36.7 mm, vias 20 -> 18
- net GND: track 82.0 -> 67.3 mm, vias 433 -> 134
- net Net-(J4-Pin_3): track 10.7 -> 0.00 mm
- net ANT_SW_CTRL: track 23.1 -> 30.3 mm
- net LORA_DIO1: track 69.3 -> 75.9 mm
- net Net-(U2-VDD3P3_CPU): track 48.2 -> 42.1 mm, vias 2 -> 4
- net D+: track 51.5 -> 56.3 mm
- net Net-(J4-Pin_20): track 8.48 -> 4.49 mm
- net Net-(U9-D): track 0.00 -> 2.34 mm
- net Net-(U17-QSTRT): track 4.60 -> 2.45 mm
- net Net-(U18-~{CTRL}/~{VDD}): track 0.00 -> 1.79 mm
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- added copper zone on F.Cu, net +3V3_2
- added copper zone on F.Cu, net Net-(U2-VDD3P3_CPU)
Other:
- board text added: "Version 0.4"
- board text removed: "Version 0.3"
