File: pcb/messenger/messenger.kicad_sch (KiCad schematic)
At the start: 57 parts, among them J1 USB_C_Receptacle_USB2.0_16P, J2 Battery, J3 Conn_Coaxial, J4 Display Connector, SW1 BOOT, SW2 EN, U10 W25Q128JVS, U14 24AA32AF-I_MS, U17 MAX17048G+T10, U2 ESP32-S3, U4 USBLC6-2SC6, U5 MCP73831-2-OT, U7 TLV76733DRVx, U8 DMG3415U-7, U9 DMG3415U-7, X1 40MHz

Commit message: pcb fixes
Parts:
- removed R8: 5.1k, Resistor_SMD:R_0603_1608Metric, symbol Device:R_US
Connections:
- net GND: now also J4.3 (Pin_3), J4.4 (Pin_4)
Changed lines of the file:
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@@
 	)
 	(junction
+		(at 384.81 78.74)
+		(diameter 0)
+		(color 0 0 0 0)
+	)
+	(junction
 		(at 160.02 41.91)
 		(diameter 0)
@@
 	(wire
 		(pts
+			(xy 384.81 78.74) (xy 384.81 85.09)
+		)
+		(stroke
+			(width 0)
+			(type default)
+		)
+	)
+	(wire
+		(pts
 			(xy 237.49 255.27) (xy 238.76 255.27)
 		)
@@
 	(wire
 		(pts
-			(xy 66.04 80.01) (xy 66.04 81.28)
+			(xy 384.81 78.74) (xy 381 78.74)
 		)
 		(stroke
@@
 	(wire
 		(pts
-			(xy 374.65 82.55) (xy 374.65 85.09)
+			(xy 66.04 80.01) (xy 66.04 81.28)
 		)
 		(stroke
@@
 	(wire
 		(pts
-			(xy 388.62 78.74) (xy 381 78.74)
+			(xy 388.62 78.74) (xy 384.81 78.74)
 		)
 		(stroke
@@
 	(wire
 		(pts
-			(xy 374.65 85.09) (xy 377.19 85.09)
-		)
-		(stroke
-			(width 0)
-			(type default)
-		)
-	)
-	(wire
-		(pts
 			(xy 223.52 96.52) (xy 228.6 96.52)
 		)
@@
 	)
 	(symbol
-		(lib_id "Device:R_US")
-		(at 381 85.09 270)
-		(unit 1)
-		(exclude_from_sim no)
-		(in_bom yes)
-		(on_board yes)
-		(dnp no)
-		(property "Reference" "R8"
-			(at 387.604 85.09 90)
-			(effects
-				(font
-					(size 1.27 1.27)
-				)
-			)
-		)
-		(property "Value" "5.1k"
-			(at 381 87.122 90)
-			(effects
-				(font
-					(size 1.27 1.27)
-				)
-			)
-		)
-		(property "Footprint" "Resistor_SMD:R_0603_1608Metric"
-			(at 380.746 86.106 90)
-			(effects
-				(font
-					(size 1.27 1.27)
-				)
-				(hide yes)
-			)
-		)
-		(property "Datasheet" "~"
-			(at 381 85.09 0)
-			(effects
-				(font
-					(size 1.27 1.27)
-				)
-				(hide yes)
-			)
-		)
-		(property "Description" "Resistor, US symbol"
-			(at 381 85.09 0)
-			(effects
-				(font
-					(size 1.27 1.27)
-				)
-				(hide yes)
-			)
-		)
-		(pin "2"
-		)
-		(pin "1"
-		)
-		(instances
-			(project "messenger"
-				(path "/3c3794b6-df2c-4cf7-82cf-83f8f28f2ff8"
-					(reference "R8")
-					(unit 1)
-				)
-			)
-		)
-	)
-	(symbol
 		(lib_id "Device:C")
 		(at 53.34 139.7 0)
@@
 					(unit 1)
 				)
-			)
-		)
-	)
-	(symbol
-		(lib_id "power:+3V3")
-		(at 374.65 82.55 0)
-		(unit 1)
-		(exclude_from_sim no)
-		(in_bom yes)
-		(on_board yes)
-		(dnp no)
-		(fields_autoplaced yes)
-		(property "Reference" "#PWR028"
-			(at 374.65 86.36 0)
-			(effects
-				(font
-					(size 1.27 1.27)
-				)
-				(hide yes)
-			)
-		)
-		(property "Value" "+3V3"
-			(at 374.65 77.47 0)
-			(effects
-				(font
-					(size 1.27 1.27)
-				)
-			)
-		)
-		(property "Footprint" ""
-			(at 374.65 82.55 0)
-			(effects
-				(font
-					(size 1.27 1.27)
-				)
-				(hide yes)
-			)
-		)
-		(property "Datasheet" ""
-			(at 374.65 82.55 0)
-			(effects
-				(font
-					(size 1.27 1.27)
-				)
-				(hide yes)
-			)
-		)
-		(property "Description" "Power symbol creates a global label with name \"+3V3\""
-			(at 374.65 82.55 0)
-			(effects
-				(font
-					(size 1.27 1.27)
-				)
-				(hide yes)
-			)
-		)
-		(pin "1"
-		)
-		(instances
-			(project "messenger"
-				(path "/3c3794b6-df2c-4cf7-82cf-83f8f28f2ff8"
-					(reference "#PWR028")
-					(unit 1)
-				)
